File: display.kicad_sch (KiCad schematic)
At the start: 40 parts, among them J301 ConnectorLCDFrontLight, J302 FPC24(0.5MM), J303 FPC10(0.5MM), Q301 2N7002, Q302 2N7002, Q303 AO3401A

Commit message: exchange backlight LED for one that is actually white and available
Parts:
- D301, D302, D303: footprint project-lib:LED_sidemount -> project-lib:LED_sidemount_C205440; LCSC C965863 -> C205440
Changed lines of the file:
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@@
     (pin "1")
   )
-  (symbol (lib_id "Device:LED") (at 78.105 62.23 90) (unit 1)
+  (symbol (lib_name "LED_1") (lib_id "Device:LED") (at 78.105 62.23 90) (unit 1)
     (in_bom yes) (on_board yes) (fields_autoplaced)
     (property "Reference" "D301" (id 0) (at 81.915 62.5474 90)
@@
       (effects (font (size 1.27 1.27)) (justify right))
     )
-    (property "Footprint" "project-lib:LED_sidemount" (id 2) (at 78.105 62.23 0)
+    (property "Footprint" "project-lib:LED_sidemount_C205440" (id 2) (at 78.105 62.23 0)
       (effects (font (size 1.27 1.27)) hide)
     )
@@
       (effects (font (size 1.27 1.27)) hide)
     )
-    (property "LCSC" "C965863" (id 5) (at 78.105 62.23 0)
+    (property "LCSC" "C205440" (id 5) (at 78.105 62.23 0)
       (effects (font (size 1.27 1.27)) hide)
     )
@@
       (effects (font (size 1.27 1.27)) (justify right))
     )
-    (property "Footprint" "project-lib:LED_sidemount" (id 2) (at 107.315 62.23 0)
+    (property "Footprint" "project-lib:LED_sidemount_C205440" (id 2) (at 107.315 62.23 0)
       (effects (font (size 1.27 1.27)) hide)
     )
@@
       (effects (font (size 1.27 1.27)) hide)
     )
-    (property "LCSC" "C965863" (id 5) (at 107.315 62.23 0)
+    (property "LCSC" "C205440" (id 5) (at 107.315 62.23 0)
       (effects (font (size 1.27 1.27)) hide)
     )
@@
       (effects (font (size 1.27 1.27)) (justify right))
     )
-    (property "Footprint" "project-lib:LED_sidemount" (id 2) (at 92.71 62.23 0)
+    (property "Footprint" "project-lib:LED_sidemount_C205440" (id 2) (at 92.71 62.23 0)
       (effects (font (size 1.27 1.27)) hide)
     )
@@
       (effects (font (size 1.27 1.27)) hide)
     )
-    (property "LCSC" "C965863" (id 5) (at 92.71 62.23 0)
-      (effects (font (size 1.27 1.27)) hide)
-    )
+    (property "LCSC" "C205440" (id 5) (at 92.71 62.23 0)
+      (effects (font (size 1.27 1.27)) hide)
+    )
